File: switch.sch (KiCad schematic (older format))
At the start: 7 parts, among them U301 LVC2G04

Commit message: Updated several part details with alternative suppliers
Parts:
- U301: Alt. Order Code (none) -> 595-SN74LVC2G04DBVR; Alt. Supplier (none) -> Mouser
Changed lines of the file:
@@
 F 8 "1287594" H 4600 2500 50  0001 C CNN "Order Code"
 F 9 "Dual Inverter Gate" H 4600 2500 50  0001 C CNN "Note"
+F 10 "Mouser" H 4600 2500 50  0001 C CNN "Alt. Supplier"
+F 11 "595-SN74LVC2G04DBVR" H 4600 2500 50  0001 C CNN "Alt. Order Code"
 	1    4600 2500
 	1    0    0    -1
