File: TCXO.sch (KiCad schematic (older format))
At the start: 37 parts, among them SW201 SW_Rotary1x6, U201 LVC1G80, U202 LVC163, U203 AUC1G04, U204 AUC2G04, U205 AUC2G04, U206 AUC2G04, X201 40.0 MHz

Commit message: Updated several part details with alternative suppliers
Parts:
- R201, R202: Part Number MCMR06X4703FTL -> MCMR06X4703FTL
- U204, U205, U206: Alt. Order Code (none) -> 595-SN74AUC2G04DCKR; Alt. Supplier (none) -> Mouser
Changed lines of the file:
@@
 F 2 "Resistor_SMD:R_0603_1608Metric" V 3430 3300 50  0001 C CNN
 F 3 "" H 3500 3300 50  0000 C CNN
-F 4 " MCMR06X4703FTL" H 3500 3300 60  0001 C CNN "Part Number"
+F 4 "MCMR06X4703FTL" H 3500 3300 60  0001 C CNN "Part Number"
 F 5 "Multicomp" H 3500 3300 60  0001 C CNN "Manufacturer"
 F 6 "0603" H 3500 3300 60  0001 C CNN "Package"
@@
 F 2 "Resistor_SMD:R_0603_1608Metric" V 3930 3300 50  0001 C CNN
 F 3 "" H 4000 3300 50  0000 C CNN
-F 4 " MCMR06X4703FTL" H 4000 3300 60  0001 C CNN "Part Number"
+F 4 "MCMR06X4703FTL" H 4000 3300 60  0001 C CNN "Part Number"
 F 5 "Multicomp" H 4000 3300 60  0001 C CNN "Manufacturer"
 F 6 "0603" H 4000 3300 60  0001 C CNN "Package"
@@
 F 8 "1606290" H 6200 4450 50  0001 C CNN "Order Code"
 F 9 "Dual Inverter Gate" H 6200 4450 50  0001 C CNN "Note"
+F 10 "Mouser" H 6200 4450 50  0001 C CNN "Alt. Supplier"
+F 11 "595-SN74AUC2G04DCKR" H 6200 4450 50  0001 C CNN "Alt. Order Code"
 	1    6200 4450
 	1    0    0    -1
@@
 F 8 "1606290" H 6200 2450 50  0001 C CNN "Order Code"
 F 9 "Dual Inverter Gate" H 6200 2450 50  0001 C CNN "Note"
+F 10 "Mouser" H 6200 2450 50  0001 C CNN "Alt. Supplier"
+F 11 "595-SN74AUC2G04DCKR" H 6200 2450 50  0001 C CNN "Alt. Order Code"
 	1    6200 2450
 	1    0    0    -1
@@
 F 8 "1606290" H 6200 7350 50  0001 C CNN "Order Code"
 F 9 "Dual Inverter Gate" H 6200 7350 50  0001 C CNN "Note"
+F 10 "Mouser" H 6200 7350 50  0001 C CNN "Alt. Supplier"
+F 11 "595-SN74AUC2G04DCKR" H 6200 7350 50  0001 C CNN "Alt. Order Code"
 	1    6200 7350
 	1    0    0    -1

Commit message: Changed output resistor from 300R to 274R to consider the impedance of the inverter output driver.
Parts:
- C201, C202, C203, C209, C213, C216, C218, C219: Description (none) -> 100nF/50V X7R 0603 ceramic capacitor; Note 100nF/50V X7R 0603 ceramic capacitor -> (none)
- C204, C205, C206, C210, C214, C215, C217, C220, C221: Description (none) -> 1nF/50V C0G/NP0 0402 ceramic capacitor; Note 1nF/50V C0G/NP0 0402 ceramic capacitor -> (none)
- C207, C208: Description (none) -> 10nF/50V X7R 0603 ceramic capacitor; Note 10nF/50V X7R 0603 ceramic capacitor -> (none)
- C211, C212: Description (none) -> 1μF/16V 0603 X7R capacitor; Note 1μF/16V 0603 X7R capacitor -> (none)
- R201, R202: Description (none) -> 470kΩ/1% 0603 resistor; Note 470kΩ/1% 0603 resistor -> (none)
- R203, R204, R205, R206, R207, R208: value 300R -> 274R; Description (none) -> 274Ω/1% 0402 resistor; Note 300Ω/1% 0402 resistor -> (none); Order Code 2447155 -> 2072862; Part Number MCWR04X3000FTL -> MCMR04X2740FTL
- SW201: Description (none) -> 6way rotary selection switch; Manufacturer (none) -> Nidec Copal; Order Code (none) -> 2854809; Package (none) -> DIP-8; Part Number (none) -> SS-10-16NP-LE; Supplier (none) -> Farnell
- U201: Description (none) -> Single D-type flip-flop positive-edge trigger; Note Single D-type flip-flop positive-edge trigger -> (none)
- U202: Description (none) -> Presettable synchronous 4-bit binary counter with synchrono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; Note Presettable synchronous 4-bit binary counter with synchrono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 -> (none)
- U203: Description (none) -> Single Inverter Gate; Note Single Inverter Gate -> (none)
- U204, U205, U206: Description (none) -> Dual Inverter Gate; Note Dual Inverter Gate -> (none)
- X201: Description (none) -> 40.0 MHz TCXO oscillator; Note 40.0 MHz TCXO oscillator -> (none)
