File: TCXOsource.kicad_pcb (KiCad board)
At the start: 2 copper layers, 70.6 x 38 mm, 76 parts, among them P101 USB_A, P102 SH2M, P103 SMA, Q401 NX3008, SW101 SW_Push, SW201 SW_Rotary1x6, U201 LVC1G80, U202 LVC163, U203 AUC1G04, U204 AUC2G04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

Commit message: Changed output resistor from 300R to 274R to consider the impedance of the inverter output driver.
Parts:
- P103: footprint jakub:SMA -> Connector_Coaxial:SMA_Amphenol_132134_Vertical
- R203, R204, R205, R206, R207, R208: value 300R -> 274R
- moved P103 0.13 mm to (218.9, 99.1)
Connections:
- P101 pad 2: (no net) -> Net-(P101-Pad2)
- P101 pad 3: (no net) -> Net-(P101-Pad3)
- P102 pad 1: +BATT -> GND
- P102 pad 2: GND -> +BATT
- SW201 pad 2: (no net) -> Net-(SW201-Pad2)
- U202 pad 15: (no net) -> Net-(U202-Pad15)
- X201 pad 1: (no net) -> Net-(X201-Pad1)
Routing:
- net +BATT: track 36.0 -> 39.3 mm
- net GND: track 300.0 -> 303.2 mm, vias 24 -> 25
Other:
- board text added: "+"
- board text added: "-"
