File: charger.sch (KiCad schematic (older format))
At the start: 24 parts, among them Q401 NX3008, U401 TLV3012, U402 MCP73831, U403 MCP1702T-3302, U404 MCP1702T-2502

Commit message: Updated several part details with alternative suppliers
Parts:
- R403: Part Number MCMR06X4703FTL -> MCMR06X4703FTL
- R404, R405, R406, R409: Part Number MCWR06X2201FTL -> MCWR06X2201FTL
- U401: Alt. Order Code (none) -> 595-TLV3012AIDBVR; Alt. Supplier (none) -> Mouser
Changed lines of the file:
@@
 F 9 "Nanopower 1.8V SOT23 comparator with voltage reference" H 2600 5200 60  0001 C CNN "Note"
 F 10 "1.74" H 2600 5200 60  0001 C CNN "Price"
+F 11 "Mouser" H 2600 5200 50  0001 C CNN "Alt. Supplier"
+F 12 "595-TLV3012AIDBVR" H 2600 5200 50  0001 C CNN "Alt. Order Code"
 	1    2600 5200
 	1    0    0    -1
@@
 F 2 "Resistor_SMD:R_0603_1608Metric" V 1880 5500 50  0001 C CNN
 F 3 "" H 1950 5500 50  0000 C CNN
-F 4 " MCMR06X4703FTL" H 1950 5500 60  0001 C CNN "Part Number"
+F 4 "MCMR06X4703FTL" H 1950 5500 60  0001 C CNN "Part Number"
 F 5 "Multicomp" H 1950 5500 60  0001 C CNN "Manufacturer"
 F 6 "0603" H 1950 5500 60  0001 C CNN "Package"
@@
 F 2 "Resistor_SMD:R_0603_1608Metric" V 2930 1950 50  0001 C CNN
 F 3 "" H 3000 1950 50  0000 C CNN
-F 4 " MCWR06X2201FTL" H 3000 1950 60  0001 C CNN "Part Number"
+F 4 "MCWR06X2201FTL" H 3000 1950 60  0001 C CNN "Part Number"
 F 5 "Multicomp" H 3000 1950 60  0001 C CNN "Manufacturer"
 F 6 "0603" H 3000 1950 60  0001 C CNN "Package"
@@
 F 2 "Resistor_SMD:R_0603_1608Metric" V 2130 5500 50  0001 C CNN
 F 3 "" H 2200 5500 50  0000 C CNN
-F 4 " MCWR06X2201FTL" H 2200 5500 60  0001 C CNN "Part Number"
+F 4 "MCWR06X2201FTL" H 2200 5500 60  0001 C CNN "Part Number"
 F 5 "Multicomp" H 2200 5500 60  0001 C CNN "Manufacturer"
 F 6 "0603" H 2200 5500 60  0001 C CNN "Package"
@@
 F 2 "Resistor_SMD:R_0603_1608Metric" V 4930 1250 50  0001 C CNN
 F 3 "" H 5000 1250 50  0000 C CNN
-F 4 " MCWR06X2201FTL" H 5000 1250 60  0001 C CNN "Part Number"
+F 4 "MCWR06X2201FTL" H 5000 1250 60  0001 C CNN "Part Number"
 F 5 "Multicomp" H 5000 1250 60  0001 C CNN "Manufacturer"
 F 6 "0603" H 5000 1250 60  0001 C CNN "Package"
@@
 F 2 "Resistor_SMD:R_0603_1608Metric" V 3130 5900 50  0001 C CNN
 F 3 "" H 3200 5900 50  0000 C CNN
-F 4 " MCWR06X2201FTL" H 3200 5900 60  0001 C CNN "Part Number"
+F 4 "MCWR06X2201FTL" H 3200 5900 60  0001 C CNN "Part Number"
 F 5 "Multicomp" H 3200 5900 60  0001 C CNN "Manufacturer"
 F 6 "0603" H 3200 5900 60  0001 C CNN "Package"

Commit message: Changed output resistor from 300R to 274R to consider the impedance of the inverter output driver.
Parts:
- C401, C403, C405: Description (none) -> 4.7μF/16V 0603 X5R capacitor; Note 4.7μF/16V 0603 X5R capacitor -> (none)
- C402: Description (none) -> 100nF/50V X7R 0603 ceramic capacitor; Note 100nF/50V X7R 0603 ceramic capacitor -> (none)
- C404, C406, C407, C408: Description (none) -> 1μF/16V 0603 X7R capacitor; Note 1μF/16V 0603 X7R capacitor -> (none)
- D401, D402: Description (none) -> Red/green dual color LED; Note Red/green dual color LED -> (none)
- Q401: Description (none) -> 30 V 230 mA P-channel Trench MOSFET; Note 30 V 230 mA P-channel Trench MOSFET -> (none)
- R401: Description (none) -> 162kΩ/1% 0603 resistor; Note 162kΩ/1% 0603 resistor -> (none)
- R402: Description (none) -> 100kΩ/1% 0603 resistor; Note 100kΩ/1% 0603 resistor -> (none)
- R403: Description (none) -> 470kΩ/1% 0603 resistor; Note 470kΩ/1% 0603 resistor -> (none)
- R404, R405, R406, R409: Description (none) -> 2.2kΩ/1% 0603 resistor; Note 2.2kΩ/1% 0603 resistor -> (none)
- R407, R408: Description (none) -> 1.5kΩ/1% 0603 resistor; Note 1.5kΩ/1% 0603 resistor -> (none)
- U401: Description (none) -> Nanopower 1.8V SOT23 comparator with voltage reference; Note Nanopower 1.8V SOT23 comparator with voltage reference -> (none)
- U402: Description (none) -> Single-cell fully integrated Li-Ion Li-Pol charger; Note Single-cell fully integrated Li-Ion Li-Pol charger -> (none)
- U403: Description (none) -> 3.3 V 250 mA Low Quiescent Current LDO Regulator; Note 3.3 V 250 mA Low Quiescent Current LDO Regulator -> (none)
- U404: Description (none) -> 2.5 V 250 mA Low Quiescent Current LDO Regulator; Note 2.5 V 250 mA Low Quiescent Current LDO Regulator -> (none)
Changed lines of the file:
@@
 EESchema Schematic File Version 4
 LIBS:TCXOsource-cache
-EELAYER 29 0
+EELAYER 30 0
 EELAYER END
 $Descr A4 11693 8268
@@
 F 7 "Farnell" H 2200 1700 60  0001 C CNN "Supplier"
 F 8 "2112741" H 2200 1700 60  0001 C CNN "Order Code"
-F 9 "4.7μF/16V 0603 X5R capacitor" H 2200 1700 60  0001 C CNN "Note"
+F 9 "4.7μF/16V 0603 X5R capacitor" H 2200 1700 60  0001 C CNN "Description"
 F 10 "0.19" H 2200 1700 60  0001 C CNN "Price"
 	1    2200 1700
@@
 F 7 "Farnell" H 2600 5200 60  0001 C CNN "Supplier"
 F 8 "2769377" H 2600 5200 60  0001 C CNN "Order Code"
-F 9 "Nanopower 1.8V SOT23 comparator with voltage reference" H 2600 5200 60  0001 C CNN "Note"
+F 9 "Nanopower 1.8V SOT23 comparator with voltage reference" H 2600 5200 60  0001 C CNN "Description"
 F 10 "1.74" H 2600 5200 60  0001 C CNN "Price"
 F 11 "Mouser" H 2600 5200 50  0001 C CNN "Alt. Supplier"
@@
 F 7 "Farnell" H 1450 4900 60  0001 C CNN "Supplier"
 F 8 "2138519" H 1450 4900 60  0001 C CNN "Order Code"
-F 9 "162kΩ/1% 0603 resistor" H 1450 4900 60  0001 C CNN "Note"
+F 9 "162kΩ/1% 0603 resistor" H 1450 4900 60  0001 C CNN "Description"
 F 10 "0.01" H 1450 4900 60  0001 C CNN "Price"
 	1    1450 4900
@@
 F 7 "Farnell" H 1450 5500 60  0001 C CNN "Supplier"
 F 8 "2447226" H 1450 5500 60  0001 C CNN "Order Code"
-F 9 "100kΩ/1% 0603 resistor" H 1450 5500 60  0001 C CNN "Note"
+F 9 "100kΩ/1% 0603 resistor" H 1450 5500 60  0001 C CNN "Description"
 F 10 "0.01" H 1450 5500 60  0001 C CNN "Price"
 F 11 "Seeed OPL" H 1450 5500 50  0001 C CNN "Alt. Supplier"
@@
 F 7 "Farnell" H 1950 5500 60  0001 C CNN "Supplier"
 F 8 "2073512" H 1950 5500 60  0001 C CNN "Order Code"
-F 9 "470kΩ/1% 0603 resistor" H 1950 5500 60  0001 C CNN "Note"
+F 9 "470kΩ/1% 0603 resistor" H 1950 5500 60  0001 C CNN "Description"
 F 10 "0.01" H 1950 5500 60  0001 C CNN "Price"
 F 11 "Seeed OPL" H 1950 5500 50  0001 C CNN "Alt. Supplier"
@@
 F 7 "Farnell" H 4500 4150 60  0001 C CNN "Supplier"
 F 8 "2112741" H 4500 4150 60  0001 C CNN "Order Code"
-F 9 "4.7μF/16V 0603 X5R capacitor" H 4500 4150 60  0001 C CNN "Note"
+F 9 "4.7μF/16V 0603 X5R capacitor" H 4500 4150 60  0001 C CNN "Description"
 F 10 "0.19" H 4500 4150 60  0001 C CNN "Price"
 	1    4500 4150
@@
 F 7 "Farnell" H 4100 2350 60  0001 C CNN "Supplier"
 F 8 "2447279" H 4100 2350 60  0001 C CNN "Order Code"
-F 9 "1.5kΩ/1% 0603 resistor" H 4100 2350 60  0001 C CNN "Note"
+F 9 "1.5kΩ/1% 0603 resistor" H 4100 2350 60  0001 C CNN "Description"
 F 10 "0.01" H 4100 2350 60  0001 C CNN "Price"
 F 11 "Seeed OPL" H 4100 2350 50  0001 C CNN "Alt. Supplier"
@@
 F 7 "Farnell" H 5700 1950 60  0001 C CNN "Supplier"
 F 8 "2112741" H 5700 1950 60  0001 C CNN "Order Code"
-F 9 "4.7μF/16V 0603 X5R capacitor" H 5700 1950 60  0001 C CNN "Note"
+F 9 "4.7μF/16V 0603 X5R capacitor" H 5700 1950 60  0001 C CNN "Description"
 F 10 "0.19" H 5700 1950 60  0001 C CNN "Price"
 	1    5700 1950
@@
 F 7 "Farnell" H 4550 1800 60  0001 C CNN "Supplier"
 F 8 "2322113" H 4550 1800 60  0001 C CNN "Order Code"
-F 9 "Red/green dual color LED" H 4550 1800 60  0001 C CNN "Note"
+F 9 "Red/green dual color LED" H 4550 1800 60  0001 C CNN "Description"
 F 10 "0.273" H 4550 1800 60  0001 C CNN "Price"
 	1    4550 1800
@@
 F 7 "Farnell" H 3600 5300 60  0001 C CNN "Supplier"
 F 8 "2322113" H 3600 5300 60  0001 C CNN "Order Code"
-F 9 "Red/green dual color LED" H 3600 5300 60  0001 C CNN "Note"
+F 9 "Red/green dual color LED" H 3600 5300 60  0001 C CNN "Description"
 F 10 "0.273" H 3600 5300 60  0001 C CNN "Price"
 	1    3600 5300
@@
 F 7 "Farnell" H 8000 5100 50  0001 C CNN "Supplier"
 F 8 "1627173" H 8000 5100 50  0001 C CNN "Order Code"
-F 9 "2.5 V 250 mA Low Quiescent Current LDO Regulator" H 8000 5100 50  0001 C CNN "Note"
+F 9 "2.5 V 250 mA Low Quiescent Current LDO Regulator" H 8000 5100 50  0001 C CNN "Description"
 	1    8000 5100
 	1    0    0    -1
@@
 F 7 "Farnell" H 6000 5100 50  0001 C CNN "Supplier"
 F 8 "1331490" H 6000 5100 50  0001 C CNN "Order Code"
-F 9 "3.3 V 250 mA Low Quiescent Current LDO Regulator" H 6000 5100 50  0001 C CNN "Note"
+F 9 "3.3 V 250 mA Low Quiescent Current LDO Regulator" H 6000 5100 50  0001 C CNN "Description"
 	1    6000 5100
 	1    0    0    -1
@@
 F 7 "Farnell" H 6500 5350 50  0001 C CNN "Supplier"
 F 8 "2768390" H 6500 5350 50  0001 C CNN "Order Code"
-F 9 "1μF/16V 0603 X7R capacitor" H 6500 5350 50  0001 C CNN "Note"
+F 9 "1μF/16V 0603 X7R capacitor" H 6500 5350 50  0001 C CNN "Description"
 F 10 "Seeed OPL" H 6500 5350 50  0001 C CNN "Alt. Supplier"
 F 11 "302010139" H 6500 5350 50  0001 C CNN "Alt. Order Code"
@@
 F 7 "Farnell" H 8500 5350 50  0001 C CNN "Supplier"
 F 8 "2768390" H 8500 5350 50  0001 C CNN "Order Code"
-F 9 "1μF/16V 0603 X7R capacitor" H 8500 5350 50  0001 C CNN "Note"
+F 9 "1μF/16V 0603 X7R capacitor" H 8500 5350 50  0001 C CNN "Description"
 F 10 "Seeed OPL" H 8500 5350 50  0001 C CNN "Alt. Supplier"
 F 11 "302010139" H 8500 5350 50  0001 C CNN "Alt. Order Code"
@@
 F 7 "Farnell" H 5500 5350 50  0001 C CNN "Supplier"
 F 8 "2768390" H 5500 5350 50  0001 C CNN "Order Code"
-F 9 "1μF/16V 0603 X7R capacitor" H 5500 5350 50  0001 C CNN "Note"
+F 9 "1μF/16V 0603 X7R capacitor" H 5500 5350 50  0001 C CNN "Description"
 F 10 "Seeed OPL" H 5500 5350 50  0001 C CNN "Alt. Supplier"
 F 11 "302010139" H 5500 5350 50  0001 C CNN "Alt. Order Code"
@@
 F 7 "Farnell" H 7500 5350 50  0001 C CNN "Supplier"
 F 8 "2768390" H 7500 5350 50  0001 C CNN "Order Code"
-F 9 "1μF/16V 0603 X7R capacitor" H 7500 5350 50  0001 C CNN "Note"
+F 9 "1μF/16V 0603 X7R capacitor" H 7500 5350 50  0001 C CNN "Description"
 F 10 "Seeed OPL" H 7500 5350 50  0001 C CNN "Alt. Supplier"
 F 11 "302010139" H 7500 5350 50  0001 C CNN "Alt. Order Code"
@@
 F 7 "Farnell" H 6500 2100 50  0001 C CNN "Supplier"
 F 8 "2069547" H 6500 2100 50  0001 C CNN "Order Code"
-F 9 "30 V 230 mA P-channel Trench MOSFET" H 6500 2100 50  0001 C CNN "Note"
+F 9 "30 V 230 mA P-channel Trench MOSFET" H 6500 2100 50  0001 C CNN "Description"
 F 10 "Seeed OPL" H 6500 2100 50  0001 C CNN "Alt. Supplier"
 F 11 "305030026" H 6500 2100 50  0001 C CNN "Alt. Order Code"
@@
 F 7 "Farnell" H 3000 1950 60  0001 C CNN "Supplier"
 F 8 "2447320" H 3000 1950 60  0001 C CNN "Order Code"
-F 9 "2.2kΩ/1% 0603 resistor" H 3000 1950 60  0001 C CNN "Note"
+F 9 "2.2kΩ/1% 0603 resistor" H 3000 1950 60  0001 C CNN "Description"
 F 10 "0.01" H 3000 1950 60  0001 C CNN "Price"
 F 11 "Seeed OPL" H 3000 1950 50  0001 C CNN "Alt. Supplier"
@@
 F 7 "Farnell" H 4100 4950 60  0001 C CNN "Supplier"
 F 8 "2447279" H 4100 4950 60  0001 C CNN "Order Code"
-F 9 "1.5kΩ/1% 0603 resistor" H 4100 4950 60  0001 C CNN "Note"
+F 9 "1.5kΩ/1% 0603 resistor" H 4100 4950 60  0001 C CNN "Description"
 F 10 "0.01" H 4100 4950 60  0001 C CNN "Price"
 F 11 "Seeed OPL" H 4100 4950 50  0001 C CNN "Alt. Supplier"
@@
 F 7 "Farnell" H 2200 5500 60  0001 C CNN "Supplier"
 F 8 "2447320" H 2200 5500 60  0001 C CNN "Order Code"
-F 9 "2.2kΩ/1% 0603 resistor" H 2200 5500 60  0001 C CNN "Note"
+F 9 "2.2kΩ/1% 0603 resistor" H 2200 5500 60  0001 C CNN "Description"
 F 10 "0.01" H 2200 5500 60  0001 C CNN "Price"
 F 11 "Seeed OPL" H 2200 5500 50  0001 C CNN "Alt. Supplier"
@@
 F 7 "Farnell" H 3500 1600 50  0001 C CNN "Supplier"
 F 8 "1840935" H 3500 1600 50  0001 C CNN "Order Code"
-F 9 "Single-cell fully integrated Li-Ion Li-Pol charger" H 3500 1600 50  0001 C CNN "Note"
+F 9 "Single-cell fully integrated Li-Ion Li-Pol charger" H 3500 1600 50  0001 C CNN "Description"
 	1    3500 1600
 	1    0    0    -1
@@
 F 7 "Farnell" H 5000 1250 60  0001 C CNN "Supplier"
 F 8 "2447320" H 5000 1250 60  0001 C CNN "Order Code"
-F 9 "2.2kΩ/1% 0603 resistor" H 5000 1250 60  0001 C CNN "Note"
+F 9 "2.2kΩ/1% 0603 resistor" H 5000 1250 60  0001 C CNN "Description"
 F 10 "0.01" H 5000 1250 60  0001 C CNN "Price"
 F 11 "Seeed OPL" H 5000 1250 50  0001 C CNN "Alt. Supplier"
@@
 F 7 "Farnell" H 3200 5900 60  0001 C CNN "Supplier"
 F 8 "2447320" H 3200 5900 60  0001 C CNN "Order Code"
-F 9 "2.2kΩ/1% 0603 resistor" H 3200 5900 60  0001 C CNN "Note"
+F 9 "2.2kΩ/1% 0603 resistor" H 3200 5900 60  0001 C CNN "Description"
 F 10 "0.01" H 3200 5900 60  0001 C CNN "Price"
 F 11 "Seeed OPL" H 3200 5900 50  0001 C CNN "Alt. Supplier"
@@
 F 7 "Farnell" H 2850 4700 60  0001 C CNN "Supplier"
 F 8 "1759122" H 2850 4700 60  0001 C CNN "Order Code"
-F 9 "100nF/50V X7R 0603 ceramic capacitor" H 2850 4700 60  0001 C CNN "Note"
+F 9 "100nF/50V X7R 0603 ceramic capacitor" H 2850 4700 60  0001 C CNN "Description"
 F 10 "0.01" H 2850 4700 60  0001 C CNN "Price"
 F 11 "Seeed OPL" H 2850 4700 50  0001 C CNN "Alt. Supplier"
